File: Board/Rev-2/rev2.brd (EAGLE design)
At the start: 150.6 x 63.2 mm, 60 parts, among them IC1 74HC595N, T1 2N3904, T2 2N3904, T3 2N3904, T4 2N3904, T5 2N3904, T6 2N3904, T7 2N3904, T8 2N3904

Commit message: Board Updates
Parts:
- removed LIMIT_REG_1, LIMIT_REG_2, LIMIT_REG_3, LIMIT_REG_4, LIMIT_REG_5, LIMIT_REG_6, LIMIT_REG_7, LIMIT_REG_8: 10 ohm, resistor:0204/7
- moved D7 8.73 mm to (96.0, 41.0)
- moved D6 8.70 mm to (119.0, 41.0)
- moved D8 8.32 mm to (73.0, 41.0)
- moved D2 5.98 mm to (120.0, 21.0)
- moved D3 5.88 mm to (97.0, 21.0)
- moved D4 4.88 mm to (73.0, 21.0)
Connections:
- removed net N$30: LIMIT_REG_1.1, T1.C
- removed net N$32: LIMIT_REG_3.1, T3.C
- removed net N$33: LIMIT_REG_2.1, T2.C
- removed net N$34: LIMIT_REG_4.1, T4.C
- removed net N$35: LIMIT_REG_8.1, T8.C
- removed net N$36: LIMIT_REG_7.1, T7.C
- removed net N$37: LIMIT_REG_6.1, T6.C
- removed net N$38: LIMIT_REG_5.1, T5.C
- net N$1: now also T5.C; no longer LIMIT_REG_5.2
- net N$2: now also T6.C; no longer LIMIT_REG_6.2
- net N$3: now also T7.C; no longer LIMIT_REG_7.2
- net N$4: now also T8.C; no longer LIMIT_REG_8.2
- net N$5: now also T4.C; no longer LIMIT_REG_4.2
- net N$6: now also T3.C; no longer LIMIT_REG_3.2
- net N$8: now also T2.C; no longer LIMIT_REG_2.2
- net N$9: now also T1.C; no longer LIMIT_REG_1.2
Routing:
- net VCC: track 415.2 -> 339.3 mm, vias 3 -> 4
- net GPIO5: track 117.0 -> 186.2 mm, vias 8 -> 3
- net ADC: track 147.8 -> 194.3 mm, vias 9 -> 7
- net RELAY5: track 129.8 -> 174.1 mm, vias 2 -> 7
- net MISO: track 192.6 -> 150.0 mm, vias 3 -> 8
- net GND: track 554.0 -> 512.7 mm, vias 0 -> 1
- net N$35: track 41.1 -> 0.00 mm, vias 1 -> 0
- net N$34: track 40.1 -> 0.00 mm, vias 1 -> 0
- net N$33: track 39.1 -> 0.00 mm, vias 2 -> 0
- net N$32: track 38.1 -> 0.00 mm
- net N$30: track 36.8 -> 0.00 mm
- net N$37: track 36.6 -> 0.00 mm
- net N$36: track 36.3 -> 0.00 mm
- net N$9: track 17.1 -> 52.3 mm
- net SHCP: track 37.3 -> 70.4 mm, vias 1 -> 0
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
Commit message: Board File Updated
Parts:
- removed GND_SWITCH, VCC_SWITCH: TOGGLE_SWITCH, Toggle Switch:TOGGLE_SWITCH
- moved PHOTO_REG 9.43 mm to (142.7, 45.4)
- moved T4 2.00 mm to (49.7, 5.85)
- moved U$2 1.41 mm to (142.7, 32.2)
- moved D5 1.00 mm to (141.0, 55.3)
- moved EXTRA_GPIO 1.00 mm to (146.0, 16.0)
Connections:
- removed net N$55: EXTRA_GPIO.12, GND_SWITCH.ON
- removed net N$56: EXTRA_GPIO.2, VCC_SWITCH.ON
- net GND: now also EXTRA_GPIO.12; no longer GND_SWITCH.IN, GND_SWITCH.OFF
- net VCC: now also EXTRA_GPIO.2; no longer VCC_SWITCH.IN, VCC_SWITCH.OFF
Routing:
- net RELAY2: track 88.1 -> 206.6 mm, vias 5 -> 12
- net 3.5V: track 310.1 -> 256.2 mm, vias 8 -> 5
- net TX: track 207.6 -> 168.5 mm, vias 4 -> 6
- net ADC: track 194.3 -> 155.5 mm, vias 7 -> 5
- net RELAY5: track 174.1 -> 136.1 mm, vias 7 -> 2
- net N$55: track 36.5 -> 0.00 mm
- net GPIO5: track 186.2 -> 151.6 mm, vias 3 -> 4
- net SHCP: track 70.4 -> 37.3 mm, vias 0 -> 1
- net STCP: track 61.4 -> 34.2 mm
- net CS0: track 159.5 -> 132.4 mm, vias 5 -> 4
- net N$1: track 78.3 -> 56.1 mm
- net RX: track 193.2 -> 171.5 mm, vias 5 -> 6
- net N$56: track 21.3 -> 0.00 mm
- net GND: track 512.7 -> 530.6 mm, vias 1 -> 2
- net SCLK: track 146.7 -> 131.1 mm, vias 4 -> 6
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